File: Battery Tester.kicad_pcb (KiCad board)
At the start: 2 copper layers, 97 x 157 mm, 172 parts, among them J1 USB-C Receptacle, J2 JST-PH, J3 FTS-107-01-X-DV-A, J5 OLED DISPLAY, J6 FLE-105-01-X-DV-A, J7 TFM-110-12-X-D-A, J8 JST-PH, Q1 IRF540N, Q2 IRF540N, SW1 Reset, SW2 BOOTSEL, SW3 RotaryEncoder_Switch, SW4 Start/Stop, SW5 Charge, SW6 Discharge, U1 RP2040, U10 TLV9001IDCK, U11 MCP4725xxx-xCH, U12 MCP4725xxx-xCH, U13 MCP4725xxx-xCH, U14 TLV9001IDCK, U15 TLV9001IDCK, U16 INA219BxD, U17 21-0168E_T822-3_MXM, U2 W25Q32JVSS, U3 USBLC6-2SC6, U4 AP2112K-3.3, U5 21-0168E_T822-3_MXM, U6 LTC4001, U7 INA219BxD, U8 TLV9001IDCK, U9 MCP4725xxx-xCH, Y1 12MHz

Commit message: More routing
Parts:
- added REF**: MountingHole_2.2mm_M2_DIN965, MountingHole:MountingHole_2.2mm_M2_DIN965, F.Cu at (107.3, 83.3)
- added REF**: MountingHole_2.2mm_M2_DIN965, MountingHole:MountingHole_2.2mm_M2_DIN965, F.Cu at (80.5, 83.3)
- added REF**: MountingHole_2.2mm_M2_DIN965, MountingHole:MountingHole_2.2mm_M2_DIN965, F.Cu at (85.5, 83.3)
- added kibuzzard-643A06C8: G***, kibuzzard-643A06C8, F.Cu at (57.4, 87.7)
- added kibuzzard-643A0700: G***, kibuzzard-643A0700, F.Cu at (50.7, 92.3)
- added kibuzzard-643A070F: G***, kibuzzard-643A070F, F.Cu at (55.5, 92.3)
- added kibuzzard-643A089C: G***, kibuzzard-643A089C, F.Cu at (81.9, 101.4)
- added kibuzzard-643A08B7: G***, kibuzzard-643A08B7, F.Cu at (81.9, 117.2)
- added kibuzzard-643A0912: G***, kibuzzard-643A0912, F.Cu at (64.6, 104.0)
- added kibuzzard-643A091C: G***, kibuzzard-643A091C, F.Cu at (93.1, 130.5)
- added kibuzzard-643A09FA: G***, kibuzzard-643A09FA, F.Cu at (64.2, 92.3)
- added kibuzzard-643A0FFF: G***, kibuzzard-643A0FFF, B.Cu at (57.6, 96.2)
- Q2: footprint Package_TO_SOT_THT:TO-220-3_Vertical -> Package_TO_SOT_THT:TO-220-3_Horizontal_TabDown
- U17, U5: value 21-0168E_T822-3_MXM -> MAX17048G
- moved R18 7.78 mm to (67.8, 68.0)
- moved R33 7.78 mm to (66.3, 68.0)
- moved U12 6.22 mm to (55.5, 96.2), turned to 90 degrees
- moved C29 6.01 mm to (55.7, 100.6), turned to 180 degrees
- moved U11 5.43 mm to (50.7, 96.1), turned to 90 degrees
- moved C28 5.42 mm to (55.7, 99.1), turned to 180 degrees
- moved J3 5.13 mm to (112.1, 94.9)
- moved R55 4.52 mm to (64.2, 98.8), turned to 90 degrees
- moved R53 4.30 mm to (124.7, 86.8)
- moved U6 4.28 mm to (58.0, 110.3)
- moved C26 4.25 mm to (52.8, 110.0)
- moved R16 4.25 mm to (52.8, 108.5)
- moved R17 4.15 mm to (63.2, 108.1)
- moved R24 4.15 mm to (63.2, 109.6)
- moved R27 4.15 mm to (63.2, 111.1)
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Connections:
- C30 pad 1: /D10 -> /D02
- C31 pad 1: /D11 -> /D01
- D8 pad 2: /D11 -> unconnected-(D8-A-Pad2)
- D9 pad 2: /D12 -> unconnected-(D9-A-Pad2)
- J5 pad 1: /SDA1 -> /SDA0
- J5 pad 2: /SCL1 -> /SCL0
- JP1 pad 1: /SDA0 -> /SDA1
- JP2 pad 2: /SCL0 -> /SCL1
- R17 pad 2: /D02 -> /D10
- R24 pad 1: /D02 -> /D10
- R24 pad 2: /D01 -> /D12
- R27 pad 1: /D00 -> /D11
- R40 pad 1: /D12 -> /D00
- R41 pad 1: /D10 -> /D02
- R43 pad 1: /D11 -> /D01
- SW3 pad S2: /D12 -> /D00
- U11 pad 6: GND -> +3V3
- U12 pad 6: +3V3 -> GND
- U16 pad 3: /SDA1 -> /SDA0
- U16 pad 4: /SCL1 -> /SCL0
- U17 pad 7: /SCL1 -> /SCL0
- U17 pad 8: /SDA1 -> /SDA0
- U5 pad 7: /SCL0 -> /SCL1
- U5 pad 8: /SDA0 -> /SDA1
- U6 pad 6: /D00 -> /D11
- U6 pad 7: /D02 -> /D10
- U7 pad 3: /SDA0 -> /SDA1
- U7 pad 4: /SCL0 -> /SCL1
Routing:
- net /SDA0: track 4.57 -> 127.1 mm, vias 0 -> 4
- net /SCL0: track 6.24 -> 121.3 mm, vias 0 -> 4
- net /SCL1: track 66.4 -> 171.4 mm, vias 1 -> 6
- net /D00: track 0.00 -> 94.8 mm, vias 0 -> 1
- net 3V3_SP: track 0.00 -> 85.9 mm, vias 0 -> 2
- net /D02: track 0.00 -> 81.0 mm, vias 0 -> 2
- net /D01: track 0.00 -> 72.2 mm, vias 0 -> 2
- net /SDA1: track 70.0 -> 139.2 mm, vias 1 -> 4
- net /D13: track 3.42 -> 48.9 mm, vias 0 -> 2
- net /D12: track 97.9 -> 61.3 mm, vias 1 -> 2
- net +3V3: track 28.2 -> 55.6 mm, vias 27 -> 38
- net /DAC1: track 0.00 -> 22.8 mm
- net /D10: track 83.1 -> 64.3 mm
- net /DAC2: track 0.00 -> 12.8 mm
- net GND: track 0.00 -> 9.95 mm, vias 9 -> 30
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- added copper zone on B.Cu, net +BATT
- added copper zone on F.Cu, net +BATT
- added copper zone on B.Cu, net BATT_2
- added copper zone on B.Cu, net BATT_SENS
- added copper zone on B.Cu, net BATT_SENS_2
- added copper zone on B.Cu, net Net-(J1-SHIELD)
- added copper zone on F.Cu, net VBUS
- removed copper zone on F.Cu, net Net-(J1-SHIELD)
Other:
- board text added: "14-APR-23"
- board text added: "Idet"
- board text added: "Prog"
- board text added: "SOLAR PANEL X/Z"
- board text removed: "12-APR-23"
