File: Battery Tester.kicad_sch (KiCad schematic)
At the start: 91 parts, among them J1 USB-C Receptacle, J2 JST-PH, J3 FLE-107-01-X-DV-A, J4 Conn_01x02, J5 OLED DISPLAY, J5 SFC-110-T2-X-D-A, J6 FLE-105-01-X-DV-A, Q1 IRF540N, SW1 1-1437565-7, SW2 BOOTSEL, SW3 RotaryEncoder_Switch, SW4 Start/Stop, SW5 Charge, SW6 Discharge, U1 RP2040, U10 TLV9001IDCK, U2 AP2112K-3.3, U3 USBLC6-2SC6, U4 W25Q32JVSS, U5 MAX17048G, U6 LTC4001, U7 INA219BxD, U8 TLV9001IDCK, U9 MCP4725xxx-xCH, Y1 12MHz

Commit message: Partial Layout Completed
Parts:
- removed FB1: 600 ohm, Inductor_SMD:L_0603_1608Metric, symbol Device:FerriteBead_Small
- removed SW1: 1-1437565-7, RP Uno:SW_1-1437565-7, symbol 1-1437565-7:1-1437565-7
- added C19, C28, C32, C35: 0.1uF, Capacitor_SMD:C_0603_1608Metric, symbol Device:C_Small
- added C27, C29, C33, C34: 10uF, Capacitor_SMD:C_0603_1608Metric, symbol Device:C_Small
- added C30, C31: 0.01uF, Capacitor_SMD:C_0603_1608Metric, symbol Device:C_Small
- added C36: 1uF, Capacitor_SMD:C_0603_1608Metric, symbol Device:C_Small
- added D10, D8, D9: Blue, LED_SMD:LED_0603_1608Metric, symbol Device:LED_Small
- added D3: WS2812B, LED_SMD:LED_WS2812B_PLCC4_5.0x5.0mm_P3.2mm, symbol LED:WS2812B
- added D6, D7: Amber, LED_SMD:LED_0603_1608Metric, symbol Device:LED_Small
- added J8: JST-PH, BatteryTester:JSTPH2, symbol Connector_Generic:Conn_01x02
- added JP1, JP2: Jumper_2_Bridged, Jumper:SolderJumper-2_P1.3mm_Bridged_RoundedPad1.0x1.5mm, symbol Jumper:Jumper_2_Bridged
- added Q2: IRF540N, Package_TO_SOT_THT:TO-220-3_Vertical, symbol Transistor_FET:IRF540N
- added R33, R40, R41, R42, R43, R44, R54: 10K, Resistor_SMD:R_0603_1608Metric, symbol Device:R_Small
- added R34: 0.04R, Resistor_SMD:R_2512_6332Metric, symbol Device:R_Small
- added R35, R36, R37, R38, R5, R50, R51, R55, R59, R60: 1K, Resistor_SMD:R_0603_1608Metric, symbol Device:R_Small
- added R39: 2K, Resistor_SMD:R_0603_1608Metric, symbol Device:R_Small
- added R5 (x3): 0, Resistor_SMD:R_0603_1608Metric, symbol Device:R_Small
- added R5 (x3): 4, Resistor_SMD:R_2816_7142Metric, symbol Device:R_Small
- added R5: 1, Resistor_SMD:R_2512_6332Metric, symbol Device:R_Small
- added R52: 0.1R, Resistor_SMD:R_2512_6332Metric, symbol Device:R_Small
- added R53: 3R, Resistor_SMD:R_2512_6332Metric, symbol Device:R_Small
- added SW1: Reset, Button_Switch_SMD:SW_SPST_B3U-1000P, symbol Switch:SW_SPST
- added TP1: SCL1_MB, TestPoint:TestPoint_Pad_D1.5mm, symbol Connector:TestPoint
- added TP2: SDA1_MB, TestPoint:TestPoint_Pad_D1.5mm, symbol Connector:TestPoint
- added TP3: SWDIO, TestPoint:TestPoint_Pad_D1.5mm, symbol Connector:TestPoint
- added TP4: SWCLK, TestPoint:TestPoint_Pad_D1.5mm, symbol Connector:TestPoint
- added U11, U12, U13: MCP4725xxx-xCH, Package_TO_SOT_SMD:SOT-23-6, symbol Analog_DAC:MCP4725xxx-xCH
- added U14, U15: TLV9001IDCK, Package_TO_SOT_SMD:SOT-353_SC-70-5, symbol Amplifier_Operational:TLV9001IDCK
- added U16: INA219BxD, Package_SO:SOIC-8_3.9x4.9mm_P1.27mm, symbol Sensor_Energy:INA219BxD
- added U17: MAX17048G, BatteryTester:MAX17048G, symbol BatteryTester:MAX17048G+T10
- C18, C21, C22, C23, C26: footprint (none) -> Capacitor_SMD:C_0603_1608Metric
- D2, D3, D4, D5: value LED_Small -> Amber; footprint (none) -> LED_SMD:LED_0603_1608Metric
- D6: footprint (none) -> LED_SMD:LED_0603_1608Metric
- HS2: footprint (none) -> BatteryTester:RAT2X38E
- J2: footprint (none) -> BatteryTester:JSTPH2
- J3: value FLE-107-01-X-DV-A -> FTS-107-01-X-DV-A; footprint batteryboard:SAMTEC_FLE-107-01-X-DV-A -> BatteryTester:SAMTEC-FTS-107-01-X-DV-A
- J5: value SFC-110-T2-X-D-A -> TFM-110-12-X-D-A; footprint mainboard:SAMTEC_SFC-110-T2-X-D-A -> BatteryTester:SAMTEC_TFM-110-12-X-D-A
- J5: footprint (none) -> Connector_PinSocket_2.54mm:PinSocket_1x04_P2.54mm_Vertical
- J6: footprint (none) -> BatteryTester:SAMTEC_FLE-105-01-X-DV-A
- L1: footprint (none) -> Inductor_SMD:L_0805_2012Metric
- R12, R13, R14, R15, R16, R26, R28, R29, R30, R31, R32: footprint (none) -> Resistor_SMD:R_0603_1608Metric
- R18: value 0.04R -> 10K; footprint Resistor_SMD:R_2512_6332Metric -> Resistor_SMD:R_0603_1608Metric
- R5: value 1 -> 4; footprint Resistor_SMD:R_0603_1608Metric -> Resistor_SMD:R_2816_7142Metric
- SW3: footprint (none) -> Rotary_Encoder:RotaryEncoder_Alps_EC11E-Switch_Vertical_H20mm
- SW4, SW5, SW6: footprint (none) -> Button_Switch_SMD:SW_SPST_B3U-1000P; symbol Switch:SW_MEC_5E -> Switch:SW_SPST
- U1: footprint RP Uno:QFN40P700X700X90-57N -> BatteryTester:IC57_RP2040
- U5: footprint 21-0168E_T822-3_MXM -> BatteryTester:MAX17048G
Connections:
- net A01 is gone; now on net 3V3_SP: U1.39 (GPIO27/ADC1)
- net +3V3: now also R12.2, R18.2, C19.1, C27.1, C28.1, C29.1, C32.1, C33.1, C35.1, D3.1 (VDD), D6.2 (A), D7.2 (A), R33.2, R39.1, R42.2, R44.2, U11.3 (VDD), U12.3 (VDD), U12.6 (A0), U13.3 (VDD), U13.6 (A0), U14.5 (V+), U15.5 (V+), U16.5 (VS); no longer R14.2
- net +BATT: now also R34.2, R53.2; no longer R18.2
- net 3V3_SP: now also Q2.2 (D)
- net A03: now also R5.1, U14.4
- net BATT_SENS: now also R34.1; no longer R18.1
- net CTG: now also R14.2, SW3.C, C19.2, C27.2, C28.2, C29.2, C30.2, C31.2, C32.2, C33.2, C35.2, C36.2, D3.3 (VSS), J8.2 (Pin_2), R35.1, R36.1, R37.1, R38.1, R40.2, R5.1, R5.1, R5.1, R5.1, R5.1, R50.1, R51.1, R54.2, R55.1, SW1.1 (A), U11.2 (VSS), U11.6 (A0), U12.2 (VSS), U13.2 (VSS), U14.2 (V-), U15.2 (V-), U16.1 (A1), U16.2 (A0), U16.6 (GND), U17.1 (CTG), U17.4 (VSS), U17.9 (PAD); no longer R12.2
- net D03: now also SW4.2 (B); no longer SW4.3 (K), SW4.4 (A)
- net D04: now also SW5.2 (B); no longer SW5.3 (K), SW5.4 (A)
- net D05: now also SW6.2 (B); no longer SW6.3 (K), SW6.4 (A)
- net D06: now also D2.2 (A)
- net D07: now also D3.2 (A)
- net D08: now also D4.2 (A)
- net D09: now also D5.2 (A)
- net D10: now also C30.1, R41.1
- net D11: now also C31.1, D8.2 (A), R43.1
- net D12: now also SW3.S2, D9.2 (A), R40.1
- net D13: now also D10.2 (A)
- net DAC1: now also U11.1 (VOUT)
- net DAC2: now also U12.1 (VOUT)
- net DBus+: now also U3.6 (I/O1); no longer U3.4 (I/O2)
- net DBus-: now also U3.4 (I/O2); no longer U3.6 (I/O1)
- net NEOPIXEL: now also D3.4 (DIN)
- net RESET: now also SW1.2 (B)
- net RXLED: now also R59.1
- net SCL0: now also R12.1, JP2.2 (B), U13.5 (SCL); no longer R14.1
- net SCL1: now also R18.1, U11.5 (SCL), U12.5 (SCL), U16.4 (SCL), U17.7 (SCL)
- net SDA0: now also JP1.1 (A), U13.4 (SDA)
- net SDA1: now also R33.1, U11.4 (SDA), U12.4 (SDA), U16.3 (SDA), U17.8 (SDA)
- net SWCLK: now also TP4.1
- net SWDIO: now also TP3.1
- net TXLED: now also R60.1
- net VBUS: now also J1.A4 (VBUS), J1.A9 (VBUS), J1.B4 (VBUS), J1.B9 (VBUS)
- net at J6.7 (Pin_7): now also JP1.2 (B)
- net at J6.8 (Pin_8): now also JP2.1 (A)
- net at R30.2, SW5.1 (A): no longer SW5.2
- net at R28.2, SW4.1 (A): no longer SW4.2
- net at R15.2: now also U3.1 (I/O1); no longer U3.3 (I/O2)
- net at SW3.A: now also R41.2, R42.1
- net at SW3.B: now also R43.2, R44.1
- net at SW3.S1: now also R39.2
- net at Q1.3 (S), R5.2, R5.2: now also R5.2, R5.2, R5.2
- net at D3.1 (K): now also R36.2
- net at D4.1 (K): now also R37.2
- net at R32.2, SW6.1 (A): no longer SW6.2
- net at R12.1: now also U3.3 (I/O2); no longer U3.1 (I/O1)
- net at D2.1 (K): now also R35.2
- net at D5.1 (K): now also R38.2
- net at U5.6 (QSTRT): now also R14.1; no longer R12.1
- net SCL1_MB: no longer names the net of J5.6 (Pin_6)
- net SCL1_MB: now also TP1.1
- net SDA1_MB: no longer names the net of J5.8 (Pin_8)
- net SDA1_MB: now also TP2.1
- new net: D9.1 (K), R51.2
- new net: C34.1, R5.1, U14.1 (+), U15.3 (-)
- new net: R5.2, R5.2, U14.3 (-)
- new net: D7.1 (K), R60.2
- new net: D10.1 (K), R55.2
- new net: D6.1 (K), R59.2
- new net: C34.2, R5.1, U15.4
- new net: Q2.1 (G), R5.2
- new net: D8.1 (K), R50.2
- new net: Q2.3 (S), R5.2, R5.2
- new net: U13.1 (VOUT), U15.1 (+)
- new net: R54.1, U17.6 (QSTRT)
- new net BATT_2: R52.2, R53.1, U16.7 (IN-)
- new net BATT_SENS_2: C36.1, J8.1 (Pin_1), R52.1, U16.8 (IN+), U17.2 (CELL), U17.3 (VDD)
Other:
- note added: "+BATT CHG LED"
- note added: "+BATT DCHG LED"
- note added: "3V3_SP DCHG LED"
- note added: "BATTERY DISCHARGER OPTION 1 CONSTANT CURRENT Enable via I2C DAC DCHRG start LED, DCHRG end LED Program Discharge Current w/ DAC"
- note added: "BATTERY DISCHARGER OPTION 2 CONSTANT LOAD Enable via I2C DAC DCHRG start LED, DCHRG end LED Program Load by sensing voltages and math"
- note added: "Battery Balancer"
- note added: "Battery Tester"
- note added: "CHG COMPLETE LED"
- note added: "CHG MODE LED"
- note added: "Connect new battery w/ CC/CL discharger to measure capacity Connect satellite batteryboard w/ CC/CL discharger to discharge Connect new battery w/ mainboard to test mainboard voltage range Connect satellite batteryboard w/ mainboard to simulate satellite operation OR Connect battery + solar panel + discharge 3V3_SP"
- note added: "DCHG COMPLETE LED"
- note added: "DCHG MODE LED"
- note added: "Fuel Gauge - I2C 0 Measure BATT_SENS and charge percent Plot voltage vs. time Powered by Battery Power - Always On"
- note added: "Max Discharge: 1.7A (OR 1C)"
- note added: "Max Discharge: 110mA"
- note added: "MosFET connected to PCB GND"
- note added: "MosFET connected to heatsink"
- note added: "Possible DNI, since we can use the first current sense to measure balancing current"
- note removed: "BATTERY DISCHARGER OPTION 1 CONSTANT CURRENT Enable via I2C DAC DCHRG start LED, DCHRG end LED - MCU detect? Program Discharge Current w/ DAC"
- note removed: "BATTERY DISCHARGER OPTION 2 CONSTANT LOAD Enable via I2C DAC DCHRG start LED, DCHRG end LED - MCU detect? Program Load by sensing voltages and math"
- note removed: "Connect new battery w/ CC/CL discharger to measure capacity Connect satellite batteryboard w/ CC/CL discharger to discharge Connect new battery w/ mainboard to test mainboard voltage range Connect satellite batteryboard w/ mainboard to simulate satellite operation"
- note removed: "Fuel Gauge - I2C 0 Measure BATT_SENS and charge percent Plot voltage vs. time Powered by Battery Power - Always On Breakout I2C? Breakout +Batt? Connect nALRT and QSTRT?"
- company: (none) -> RExLab Carnegie Mellon University
- title: (none) -> PyCubed-Mini
- moved on the sheet: C21, C22, C23, D2, D3, D4, D5, HS2, J5, J6, Q1, R12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

Commit message: More routing
Parts:
- Q2: footprint Package_TO_SOT_THT:TO-220-3_Vertical -> Package_TO_SOT_THT:TO-220-3_Horizontal_TabDown
Connections:
- net +3V3: now also U11.6 (A0); no longer U12.6 (A0)
- net CTG: now also U12.6 (A0); no longer U11.6 (A0)
- net D00: now also R40.1, SW3.S2; no longer R7.1, U6.6 (~{EN})
- net D01: now also C31.1, R43.1; no longer R7.2
- net D02: now also C30.1, R41.1; no longer R7.1, R7.2, U6.7 (~{CHRG})
- net D10: now also R7.1, R7.2, U6.7 (~{CHRG}); no longer C30.1, R41.1
- net D11: now also R7.1, U6.6 (~{EN}); no longer C31.1, D8.2 (A), R43.1
- net D12: now also R7.2; no longer D9.2 (A), R40.1, SW3.S2
- net SCL0: now also J5.2 (Pin_2), U16.4 (SCL), U17.7 (SCL); no longer JP2.2 (B), U5.7 (SCL), U7.4 (SCL)
- net SCL1: now also JP2.2 (B), U5.7 (SCL), U7.4 (SCL); no longer J5.2 (Pin_2), U16.4 (SCL), U17.7 (SCL)
- net SDA0: now also J5.1 (Pin_1), U16.3 (SDA), U17.8 (SDA); no longer JP1.1 (A), U5.8 (SDA), U7.3 (SDA)
- net SDA1: now also JP1.1 (A), U5.8 (SDA), U7.3 (SDA); no longer J5.1 (Pin_1), U16.3 (SDA), U17.8 (SDA)
Changed lines of the file:
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@@
     (stroke (width 0) (type default))
   )
-  (wire (pts (xy 456.692 265.049) (xy 471.551 265.049))
+  (wire (pts (xy 395.859 265.049) (xy 410.718 265.049))
     (stroke (width 0) (type default))
   )
@@
     (stroke (width 0) (type default))
   )
-  (wire (pts (xy 456.692 263.144) (xy 456.692 265.049))
+  (wire (pts (xy 395.859 263.144) (xy 395.859 265.049))
     (stroke (width 0) (type default))
   )
@@
     (stroke (width 0) (type default))
   )
-  (wire (pts (xy 405.638 265.049) (xy 410.718 265.049))
+  (wire (pts (xy 466.471 265.049) (xy 471.551 265.049))
     (stroke (width 0) (type default))
   )
@@
     (stroke (width 0) (type default))
   )
-  (wire (pts (xy 405.638 267.716) (xy 405.638 265.049))
+  (wire (pts (xy 466.471 267.716) (xy 466.471 265.049))
     (stroke (width 0) (type default))
   )
@@
     (effects (font (size 1.27 1.27)) (justify left bottom))
   )
-  (label "SDA0" (at 542.163 187.071 0) (fields_autoplaced)
+  (label "SDA1" (at 542.163 187.071 0) (fields_autoplaced)
     (effects (font (size 1.27 1.27)) (justify left bottom))
   )
@@
     (effects (font (size 1.27 1.27)) (justify left bottom))
   )
+  (label "D08" (at -30.099 151.892 180) (fields_autoplaced)
+    (effects (font (size 1.27 1.27)) (justify right bottom))
+  )
   (label "SCK" (at 116.205 119.761 180) (fields_autoplaced)
     (effects (font (size 1.27 1.27)) (justify right bottom))
@@
     (effects (font (size 1.27 1.27)) (justify left bottom))
   )
-  (label "D11" (at 455.549 112.395 0) (fields_autoplaced)
+  (label "D01" (at 455.549 112.395 0) (fields_autoplaced)
     (effects (font (size 1.27 1.27)) (justify left bottom))
   )
@@
     (effects (font (size 1.27 1.27)) (justify left bottom))
   )
-  (label "SCL1" (at 477.901 75.946 0) (fields_autoplaced)
+  (label "SCL0" (at 477.901 75.946 0) (fields_autoplaced)
     (effects (font (size 1.27 1.27)) (justify left bottom))
   )
@@
     (effects (font (size 1.27 1.27)) (justify left bottom))
   )
-  (label "SCL1" (at 731.266 51.181 180) (fields_autoplaced)
+  (label "SCL0" (at 731.266 51.181 180) (fields_autoplaced)
     (effects (font (size 1.27 1.27)) (justify right bottom))
   )
@@
     (effects (font (size 1.27 1.27)) (justify right bottom))
   )
-  (label "D09" (at -30.226 161.798 180) (fields_autoplaced)
-    (effects (font (size 1.27 1.27)) (justify right bottom))
-  )
   (label "SWDIO" (at 51.689 84.201 0) (fields_autoplaced)
     (effects (font (size 1.27 1.27)) (justify left bottom))
@@
     (effects (font (size 1.27 1.27)) (justify right bottom))
   )
-  (label "D12" (at 62.611 364.998 180) (fields_autoplaced)
-    (effects (font (size 1.27 1.27)) (justify right bottom))
-  )
   (label "QSPI_DATA3" (at 116.205 86.741 180) (fields_autoplaced)
     (effects (font (size 1.27 1.27)) (justify right bottom))
   )
-  (label "D01" (at 476.123 205.867 180) (fields_autoplaced)
+  (label "D10" (at 476.123 209.169 180) (fields_autoplaced)
     (effects (font (size 1.27 1.27)) (justify right bottom))
   )
@@
     (effects (font (size 1.27 1.27)) (justify left bottom))
   )
-  (label "SCL0" (at 593.09 187.071 180) (fields_autoplaced)
+  (label "SCL1" (at 593.09 187.071 180) (fields_autoplaced)
     (effects (font (size 1.27 1.27)) (justify right bottom))
   )
@@
     (effects (font (size 1.27 1.27)) (justify left bottom))
   )
-  (label "D00" (at 412.115 175.768 0) (fields_autoplaced)
+  (label "D11" (at 412.115 175.768 0) (fields_autoplaced)
     (effects (font (size 1.27 1.27)) (justify left bottom))
   )
@@
     (effects (font (size 1.27 1.27)) (justify right bottom))
   )
-  (label "SDA1" (at 731.266 47.371 180) (fields_autoplaced)
+  (label "SDA0" (at 731.266 47.371 180) (fields_autoplaced)
     (effects (font (size 1.27 1.27)) (justify right bottom))
   )
@@
     (effects (font (size 1.27 1.27)) (justify left bottom))
   )
-  (label "SCL0" (at 450.088 59.817 180) (fields_autoplaced)
+  (label "SCL1" (at 450.088 59.817 180) (fields_autoplaced)
     (effects (font (size 1.27 1.27)) (justify right bottom))
   )
-  (label "D10" (at 455.549 107.315 0) (fields_autoplaced)
+  (label "D02" (at 455.549 107.315 0) (fields_autoplaced)
     (effects (font (size 1.27 1.27)) (justify left bottom))
   )
@@
     (effects (font (size 1.27 1.27)) (justify right bottom))
   )
-  (label "SDA0" (at 369.062 56.515 180) (fields_autoplaced)
+  (label "SDA1" (at 369.062 56.515 180) (fields_autoplaced)
     (effects (font (size 1.27 1.27)) (justify right bottom))
   )
@@
     (effects (font (size 1.27 1.27)) (justify right bottom))
   )
-  (label "D08" (at -30.099 151.892 180) (fields_autoplaced)
-    (effects (font (size 1.27 1.27)) (justify right bottom))
-  )
   (label "D10" (at 45.339 127.381 0) (fields_autoplaced)
     (effects (font (size 1.27 1.27)) (justify left bottom))
   )
-  (label "SCL0" (at 369.062 60.325 180) (fields_autoplaced)
+  (label "SCL1" (at 369.062 60.325 180) (fields_autoplaced)
     (effects (font (size 1.27 1.27)) (justify right bottom))
   )
@@
     (effects (font (size 1.27 1.27)) (justify left bottom))
   )
-  (label "D02" (at 476.123 209.169 180) (fields_autoplaced)
+  (label "D12" (at 476.123 205.867 180) (fields_autoplaced)
     (effects (font (size 1.27 1.27)) (justify right bottom))
   )
-  (label "SCL1" (at 654.431 51.435 180) (fields_autoplaced)
+  (label "SCL0" (at 654.431 51.435 180) (fields_autoplaced)
     (effects (font (size 1.27 1.27)) (justify right bottom))
   )
@@
     (effects (font (size 1.27 1.27)) (justify right bottom))
   )
-  (label "D12" (at 504.063 112.395 180) (fields_autoplaced)
+  (label "D00" (at 504.063 112.395 180) (fields_autoplaced)
     (effects (font (size 1.27 1.27)) (justify right bottom))
   )
@@
     (effects (font (size 1.27 1.27)) (justify left bottom))
   )
-  (label "SDA1" (at 654.431 48.895 180) (fields_autoplaced)
+  (label "D09" (at -30.226 161.798 180) (fields_autoplaced)
     (effects (font (size 1.27 1.27)) (justify right bottom))
   )
-  (label "QSPI_DATA0" (at 214.63 136.652 180) (fields_autoplaced)
+  (label "SDA0" (at 654.431 48.895 180) (fields_autoplaced)
     (effects (font (size 1.27 1.27)) (justify right bottom))
   )
-  (label "D11" (at -64.897 364.363 180) (fields_autoplaced)
+  (label "QSPI_DATA0" (at 214.63 136.652 180) (fields_autoplaced)
     (effects (font (size 1.27 1.27)) (justify right bottom))
   )
@@
     (effects (font (size 1.27 1.27)) (justify left bottom))
   )
-  (label "SDA0" (at 450.088 57.277 180) (fields_autoplaced)
+  (label "SDA1" (at 450.088 57.277 180) (fields_autoplaced)
     (effects (font (size 1.27 1.27)) (justify right bottom))
   )
@@
     (effects (font (size 1.27 1.27)) (justify right bottom))
   )
-  (label "SDA1" (at 477.901 73.406 0) (fields_autoplaced)
+  (label "SDA0" (at 477.901 73.406 0) (fields_autoplaced)
     (effects (font (size 1.27 1.27)) (justify left bottom))
   )
@@
     )
   )
-  (symbol (lib_id "power:+3V3") (at 456.692 263.144 0) (unit 1)
+  (symbol (lib_id "power:+3V3") (at 395.859 263.144 0) (unit 1)
     (in_bom yes) (on_board yes) (dnp no)
-    (property "Reference" "#PWR0145" (at 456.692 266.954 0)
+    (property "Reference" "#PWR0145" (at 395.859 266.954 0)
       (effects (font (size 1.27 1.27)) hide)
     )
-    (property "Value" "+3V3" (at 456.692 259.461 0)
+    (property "Value" "+3V3" (at 395.859 259.461 0)
       (effects (font (size 1.27 1.27)))
     )
-    (property "Footprint" "" (at 456.692 263.144 0)
+    (property "Footprint" "" (at 395.859 263.144 0)
       (effects (font (size 1.27 1.27)) hide)
     )
-    (property "Datasheet" "" (at 456.692 263.144 0)
+    (property "Datasheet" "" (at 395.859 263.144 0)
       (effects (font (size 1.27 1.27)) hide)
     )
@@
     )
   )
-  (symbol (lib_id "power:GND") (at 405.638 267.716 0) (unit 1)
+  (symbol (lib_id "power:GND") (at 466.471 267.716 0) (unit 1)
     (in_bom yes) (on_board yes) (dnp no)
-    (property "Reference" "#PWR0138" (at 405.638 274.066 0)
+    (property "Reference" "#PWR0138" (at 466.471 274.066 0)
       (effects (font (size 1.27 1.27)) hide)
     )
-    (property "Value" "GND" (at 405.638 271.526 0)
+    (property "Value" "GND" (at 466.471 271.526 0)
       (effects (font (size 1.27 1.27)))
     )
-    (property "Footprint" "" (at 405.638 267.716 0)
+    (property "Footprint" "" (at 466.471 267.716 0)
       (effects (font (size 1.27 1.27)) hide)
     )
-    (property "Datasheet" "" (at 405.638 267.716 0)
+    (property "Datasheet" "" (at 466.471 267.716 0)
       (effects (font (size 1.27 1.27)) hide)
     )
@@
       (effects (font (size 1.27 1.27)) (justify left))
     )
-    (property "Footprint" "Package_TO_SOT_THT:TO-220-3_Vertical" (at -1.905 284.353 0)
+    (property "Footprint" "Package_TO_SOT_THT:TO-220-3_Horizontal_TabDown" (at -1.905 284.353 0)
       (effects (font (size 1.27 1.27) italic) (justify left) hide)
     )

Commit message: Finished Routing
Parts:
- added TP5: A01, TestPoint:TestPoint_Pad_D1.5mm, symbol Connector:TestPoint
- added TP6: BATT_SENS, TestPoint:TestPoint_Pad_D1.5mm, symbol Connector:TestPoint
- added TP7, TP9: GND, TestPoint:TestPoint_Pad_D1.5mm, symbol Connector:TestPoint
- added TP8: BATT_SENS_2, TestPoint:TestPoint_Pad_D1.5mm, symbol Connector:TestPoint
- HS2: symbol Mechanical:Heatsink_Pad -> Mechanical:Heatsink_Pad_2Pin
- J3: value FTS-107-01-X-DV-A -> FLE-107-01-X-DV-A; footprint BatteryTester:SAMTEC-FTS-107-01-X-DV-A -> BatteryTester:SAMTEC_FLE-107-01-X-DV-A
Connections:
- net USB_HOSTEN is gone; now on net D14: U1.28 (GPIO17)
- net 3V3_SP: now also U1.38 (GPIO26/ADC0); no longer U1.39 (GPIO27/ADC1)
- net A02: now also R5.1, U10.4
- net BATT_SENS: now also TP6.1
- net BATT_SENS_2: now also TP8.1
- net CTG: now also HS2.2, TP7.1, TP9.1
- net D14: now reaches D9.2 (A)
- net D15: now reaches U1.35 (GPIO23)
- net D15: now also D8.2 (A)
- removed net A00: R5.1, U1.38 (GPIO26/ADC0), U10.4
- new net A01: TP5.1, U1.39 (GPIO27/ADC1)
- no-connect marks 31 -> 30
Other:
- note added: "I2C0 0x62"
- note added: "I2C0 0x63"
